Commit message: feat: add local Raptor control demo, decision models and verified evidence

File: src/raptor_description/urdf/raptor.urdf.xacro (robot description, xacro)
@@ -3,4 +3,47 @@
   xmlns:xacro="http://www.ros.org/wiki/xacro"
   name="raptor">
+  <!-- Bench fixture is explicitly opt-in and never a standing validation. -->
+  <xacro:arg name="test_fixture" default="false"/>
+  <xacro:arg name="detailed_visuals" default="false"/>
+  <xacro:arg name="sensors" default="false"/>
+  <xacro:if value="$(arg sensors)">
+    <gazebo reference="base_link">
+      <sensor name="body_imu" type="imu">
+        <always_on>true</always_on><update_rate>50</update_rate>
+        <topic>/raptor/imu</topic>
+      </sensor>
+      <sensor name="front_rgbd" type="rgbd_camera">
+        <pose>0.42 0 0.04 0 0 0</pose>
+        <always_on>true</always_on><update_rate>5</update_rate>
+        <topic>/raptor/camera</topic>
+        <camera>
+          <horizontal_fov>1.05</horizontal_fov>
+          <image><width>320</width><height>240</height><format>R8G8B8</format></image>
+          <clip><near>0.05</near><far>20</far></clip>
+          <depth_camera><clip><near>0.05</near><far>20</far></clip></depth_camera>
+        </camera>
+      </sensor>
+    </gazebo>
+    <xacro:macro name="foot_contact" params="side">
+      <gazebo reference="${side}_foot_link">
+        <sensor name="${side}_foot_contact" type="contact">
+          <always_on>true</always_on><update_rate>50</update_rate>
+          <topic>/raptor/${side}_foot/contact</topic>
+          <contact>
+            <collision>${side}_foot_link_collision</collision>
+            <topic>/raptor/${side}_foot/contact</topic>
+          </contact>
+        </sensor>
+      </gazebo>
+    </xacro:macro>
+    <xacro:foot_contact side="left"/><xacro:foot_contact side="right"/>
+  </xacro:if>
+  <xacro:if value="$(arg test_fixture)">
+    <link name="world"/>
+    <joint name="test_fixture_joint" type="fixed">
+      <parent link="world"/><child link="base_root"/>
+      <origin xyz="0 0 0.25"/>
+    </joint>
+  </xacro:if>
     <!-- Dummy root link for KDL -->
   <link name="base_root"/>
@@ -16,5 +59,5 @@
   <link name="base_link">
     <!-- 화면에 보이는 외형 -->
-    <visual>
+    <xacro:unless value="$(arg detailed_visuals)"><visual>
       <origin xyz="0 0 0" rpy="0 0 0"/>
       <geometry>
@@ -24,5 +67,13 @@
         <color rgba="0.35 0.37 0.40 1.0"/>
       </material>
-    </visual>
+    </visual></xacro:unless>
+    <xacro:if value="$(arg detailed_visuals)">
+      <visual><geometry><mesh filename="package://raptor_description/meshes/raptor/base_link__graphite.dae"/></geometry><material name="raptor_graphite"><color rgba="0.065 0.075 0.085 1"/></material></visual>
+      <visual><geometry><mesh filename="package://raptor_description/meshes/raptor/base_link__titanium.dae"/></geometry><material name="raptor_titanium"><color rgba="0.36 0.4 0.43 1"/></material></visual>
+      <visual><geometry><mesh filename="package://raptor_description/meshes/raptor/base_link__ivory.dae"/></geometry><material name="raptor_ivory"><color rgba="0.72 0.72 0.65 1"/></material></visual>
+      <visual><geometry><mesh filename="package://raptor_description/meshes/raptor/base_link__copper.dae"/></geometry><material name="raptor_copper"><color rgba="0.66 0.29 0.08 1"/></material></visual>
+      <visual><geometry><mesh filename="package://raptor_description/meshes/raptor/base_link__rubber.dae"/></geometry><material name="raptor_rubber"><color rgba="0.025 0.028 0.032 1"/></material></visual>
+      <visual><geometry><mesh filename="package://raptor_description/meshes/raptor/base_link__lens.dae"/></geometry><material name="raptor_lens"><color rgba="0.05 0.26 0.33 1"/></material></visual>
+    </xacro:if>
     <!-- Gazebo가 충돌 계산할 때 사용하는 모양 -->
     <collision>
@@ -50,5 +101,5 @@
     <!-- ========================================= -->
     <link name="left_hip_roll_link">
-    <visual>
+    <xacro:unless value="$(arg detailed_visuals)"><visual>
       <origin xyz="0 0 -0.06" rpy="0 0 0"/>
       <geometry>
@@ -58,5 +109,10 @@
         <color rgba="0.15 0.16 0.18 1.0"/>
       </material>
-    </visual>
+    </visual></xacro:unless>
+    <xacro:if value="$(arg detailed_visuals)">
+      <visual><geometry><mesh filename="package://raptor_description/meshes/raptor/left_hip_roll_link__graphite.dae"/></geometry><material name="raptor_graphite"><color rgba="0.065 0.075 0.085 1"/></material></visual>
+      <visual><geometry><mesh filename="package://raptor_description/meshes/raptor/left_hip_roll_link__titanium.dae"/></geometry><material name="raptor_titanium"><color rgba="0.36 0.4 0.43 1"/></material></visual>
+      <visual><geometry><mesh filename="package://raptor_description/meshes/raptor/left_hip_roll_link__ivory.dae"/></geometry><material name="raptor_ivory"><color rgba="0.72 0.72 0.65 1"/></material></visual>
+    </xacro:if>
     <collision>
       <origin xyz="0 0 -0.06" rpy="0 0 0"/>
@@ -96,5 +152,5 @@
   <!-- ========================================= -->
   <link name="left_thigh_link">
-    <visual>
+    <xacro:unless value="$(arg detailed_visuals)"><visual>
       <!-- 관절에서 아래쪽으로 허벅지가 내려감 -->
       <origin xyz="0 0 -0.16" rpy="0 0 0"/>
@@ -105,5 +161,11 @@
         <color rgba="0.55 0.57 0.60 1.0"/>
       </material>
-    </visual>
+    </visual></xacro:unless>
+    <xacro:if value="$(arg detailed_visuals)">
+      <visual><geometry><mesh filename="package://raptor_description/meshes/raptor/left_thigh_link__graphite.dae"/></geometry><material name="raptor_graphite"><color rgba="0.065 0.075 0.085 1"/></material></visual>
+      <visual><geometry><mesh filename="package://raptor_description/meshes/raptor/left_thigh_link__titanium.dae"/></geometry><material name="raptor_titanium"><color rgba="0.36 0.4 0.43 1"/></material></visual>
+      <visual><geometry><mesh filename="package://raptor_description/meshes/raptor/left_thigh_link__ivory.dae"/></geometry><material name="raptor_ivory"><color rgba="0.72 0.72 0.65 1"/></material></visual>
+      <visual><geometry><mesh filename="package://raptor_description/meshes/raptor/left_thigh_link__copper.dae"/></geometry><material name="raptor_copper"><color rgba="0.66 0.29 0.08 1"/></material></visual>
+    </xacro:if>
     <collision>
       <origin xyz="0 0 -0.16" rpy="0 0 0"/>
@@ -143,5 +205,5 @@
   <!-- ========================================= -->
   <link name="left_shin_link">
-    <visual>
+    <xacro:unless value="$(arg detailed_visuals)"><visual>
       <!-- 무릎 아래로 종아리가 내려감 -->
       <origin xyz="0 0 -0.15" rpy="0 0 0"/>
@@ -152,5 +214,10 @@
         <color rgba="0.42 0.44 0.47 1.0"/>
       </material>
-    </visual>
+    </visual></xacro:unless>
+    <xacro:if value="$(arg detailed_visuals)">
+      <visual><geometry><mesh filename="package://raptor_description/meshes/raptor/left_shin_link__graphite.dae"/></geometry><material name="raptor_graphite"><color rgba="0.065 0.075 0.085 1"/></material></visual>
+      <visual><geometry><mesh filename="package://raptor_description/meshes/raptor/left_shin_link__titanium.dae"/></geometry><material name="raptor_titanium"><color rgba="0.36 0.4 0.43 1"/></material></visual>
+      <visual><geometry><mesh filename="package://raptor_description/meshes/raptor/left_shin_link__ivory.dae"/></geometry><material name="raptor_ivory"><color rgba="0.72 0.72 0.65 1"/></material></visual>
+    </xacro:if>
     <collision>
       <origin xyz="0 0 -0.15" rpy="0 0 0"/>
@@ -193,5 +260,5 @@
   <!-- ========================================= -->
   <link name="left_foot_link">
-    <visual>
+    <xacro:unless value="$(arg detailed_visuals)"><visual>
       <!-- 발목 기준으로 발을 약간 앞으로 배치 -->
       <origin xyz="0.06 0 -0.03" rpy="0 0 0"/>
@@ -202,5 +269,11 @@
         <color rgba="0.12 0.13 0.15 1.0"/>
       </material>
-    </visual>
+    </visual></xacro:unless>
+    <xacro:if value="$(arg detailed_visuals)">
+      <visual><geometry><mesh filename="package://raptor_description/meshes/raptor/left_foot_link__graphite.dae"/></geometry><material name="raptor_graphite"><color rgba="0.065 0.075 0.085 1"/></material></visual>
+      <visual><geometry><mesh filename="package://raptor_description/meshes/raptor/left_foot_link__titanium.dae"/></geometry><material name="raptor_titanium"><color rgba="0.36 0.4 0.43 1"/></material></visual>
+      <visual><geometry><mesh filename="package://raptor_description/meshes/raptor/left_foot_link__ivory.dae"/></geometry><material name="raptor_ivory"><color rgba="0.72 0.72 0.65 1"/></material></visual>
+      <visual><geometry><mesh filename="package://raptor_description/meshes/raptor/left_foot_link__rubber.dae"/></geometry><material name="raptor_rubber"><color rgba="0.025 0.028 0.032 1"/></material></visual>
+    </xacro:if>
     <collision>
       <origin xyz="0.06 0 -0.03" rpy="0 0 0"/>
@@ -241,5 +314,5 @@
   <!-- 1. RIGHT HIP ROLL LINK -->
   <link name="right_hip_roll_link">
-    <visual>
+    <xacro:unless value="$(arg detailed_visuals)"><visual>
       <origin xyz="0 0 -0.06" rpy="0 0 0"/>
       <geometry>
@@ -249,5 +322,10 @@
         <color rgba="0.15 0.16 0.18 1.0"/>
       </material>
-    </visual>
+    </visual></xacro:unless>
+    <xacro:if value="$(arg detailed_visuals)">
+      <visual><geometry><mesh filename="package://raptor_description/meshes/raptor/right_hip_roll_link__graphite.dae"/></geometry><material name="raptor_graphite"><color rgba="0.065 0.075 0.085 1"/></material></visual>
+      <visual><geometry><mesh filename="package://raptor_description/meshes/raptor/right_hip_roll_link__titanium.dae"/></geometry><material name="raptor_titanium"><color rgba="0.36 0.4 0.43 1"/></material></visual>
+      <visual><geometry><mesh filename="package://raptor_description/meshes/raptor/right_hip_roll_link__ivory.dae"/></geometry><material name="raptor_ivory"><color rgba="0.72 0.72 0.65 1"/></material></visual>
+    </xacro:if>
     <collision>
       <origin xyz="0 0 -0.06" rpy="0 0 0"/>
@@ -286,5 +364,5 @@
   <!-- 2. RIGHT HIP PITCH + THIGH -->
   <link name="right_thigh_link">
-    <visual>
+    <xacro:unless value="$(arg detailed_visuals)"><visual>
       <origin xyz="0 0 -0.16" rpy="0 0 0"/>
       <geometry>
@@ -294,5 +372,11 @@
         <color rgba="0.55 0.57 0.60 1.0"/>
       </material>
-    </visual>
+    </visual></xacro:unless>
+    <xacro:if value="$(arg detailed_visuals)">
+      <visual><geometry><mesh filename="package://raptor_description/meshes/raptor/right_thigh_link__graphite.dae"/></geometry><material name="raptor_graphite"><color rgba="0.065 0.075 0.085 1"/></material></visual>
+      <visual><geometry><mesh filename="package://raptor_description/meshes/raptor/right_thigh_link__titanium.dae"/></geometry><material name="raptor_titanium"><color rgba="0.36 0.4 0.43 1"/></material></visual>
+      <visual><geometry><mesh filename="package://raptor_description/meshes/raptor/right_thigh_link__ivory.dae"/></geometry><material name="raptor_ivory"><color rgba="0.72 0.72 0.65 1"/></material></visual>
+      <visual><geometry><mesh filename="package://raptor_description/meshes/raptor/right_thigh_link__copper.dae"/></geometry><material name="raptor_copper"><color rgba="0.66 0.29 0.08 1"/></material></visual>
+    </xacro:if>
     <collision>
       <origin xyz="0 0 -0.16" rpy="0 0 0"/>
@@ -327,5 +411,5 @@
   <!-- 3. RIGHT KNEE PITCH + SHIN -->
   <link name="right_shin_link">
-    <visual>
+    <xacro:unless value="$(arg detailed_visuals)"><visual>
       <origin xyz="0 0 -0.15" rpy="0 0 0"/>
       <geometry>
@@ -335,5 +419,10 @@
         <color rgba="0.42 0.44 0.47 1.0"/>
       </material>
-    </visual>
+    </visual></xacro:unless>
+    <xacro:if value="$(arg detailed_visuals)">
+      <visual><geometry><mesh filename="package://raptor_description/meshes/raptor/right_shin_link__graphite.dae"/></geometry><material name="raptor_graphite"><color rgba="0.065 0.075 0.085 1"/></material></visual>
+      <visual><geometry><mesh filename="package://raptor_description/meshes/raptor/right_shin_link__titanium.dae"/></geometry><material name="raptor_titanium"><color rgba="0.36 0.4 0.43 1"/></material></visual>
+      <visual><geometry><mesh filename="package://raptor_description/meshes/raptor/right_shin_link__ivory.dae"/></geometry><material name="raptor_ivory"><color rgba="0.72 0.72 0.65 1"/></material></visual>
+    </xacro:if>
     <collision>
       <origin xyz="0 0 -0.15" rpy="0 0 0"/>
@@ -367,5 +456,5 @@
   <!-- 4. RIGHT ANKLE PITCH + FOOT -->
   <link name="right_foot_link">
-    <visual>
+    <xacro:unless value="$(arg detailed_visuals)"><visual>
       <origin xyz="0.06 0 -0.03" rpy="0 0 0"/>
       <geometry>
@@ -375,5 +464,11 @@
         <color rgba="0.12 0.13 0.15 1.0"/>
       </material>
-    </visual>
+    </visual></xacro:unless>
+    <xacro:if value="$(arg detailed_visuals)">
+      <visual><geometry><mesh filename="package://raptor_description/meshes/raptor/right_foot_link__graphite.dae"/></geometry><material name="raptor_graphite"><color rgba="0.065 0.075 0.085 1"/></material></visual>
+      <visual><geometry><mesh filename="package://raptor_description/meshes/raptor/right_foot_link__titanium.dae"/></geometry><material name="raptor_titanium"><color rgba="0.36 0.4 0.43 1"/></material></visual>
+      <visual><geometry><mesh filename="package://raptor_description/meshes/raptor/right_foot_link__ivory.dae"/></geometry><material name="raptor_ivory"><color rgba="0.72 0.72 0.65 1"/></material></visual>
+      <visual><geometry><mesh filename="package://raptor_description/meshes/raptor/right_foot_link__rubber.dae"/></geometry><material name="raptor_rubber"><color rgba="0.025 0.028 0.032 1"/></material></visual>
+    </xacro:if>
     <collision>
       <origin xyz="0.06 0 -0.03" rpy="0 0 0"/>
@@ -412,5 +507,5 @@
   <!-- 몸통 뒤쪽에서 좌우로 회전하는 꼬리 베이스 -->
   <link name="tail_yaw_link">
-    <visual>
+    <xacro:unless value="$(arg detailed_visuals)"><visual>
       <!-- 관절 기준 뒤쪽(-X)으로 꼬리 베이스가 뻗음 -->
       <origin xyz="-0.08 0 0" rpy="0 0 0"/>
@@ -421,5 +516,10 @@
         <color rgba="0.18 0.19 0.21 1.0"/>
       </material>
-    </visual>
+    </visual></xacro:unless>
+    <xacro:if value="$(arg detailed_visuals)">
+      <visual><geometry><mesh filename="package://raptor_description/meshes/raptor/tail_yaw_link__graphite.dae"/></geometry><material name="raptor_graphite"><color rgba="0.065 0.075 0.085 1"/></material></visual>
+      <visual><geometry><mesh filename="package://raptor_description/meshes/raptor/tail_yaw_link__titanium.dae"/></geometry><material name="raptor_titanium"><color rgba="0.36 0.4 0.43 1"/></material></visual>
+      <visual><geometry><mesh filename="package://raptor_description/meshes/raptor/tail_yaw_link__ivory.dae"/></geometry><material name="raptor_ivory"><color rgba="0.72 0.72 0.65 1"/></material></visual>
+    </xacro:if>
     <collision>
       <origin xyz="-0.08 0 0" rpy="0 0 0"/>
@@ -457,5 +557,5 @@
   <!-- 꼬리를 위아래로 움직이는 관절 -->
   <link name="tail_link">
-    <visual>
+    <xacro:unless value="$(arg detailed_visuals)"><visual>
       <!-- Pitch 관절에서 뒤쪽으로 0.5m 뻗는 꼬리 -->
       <origin xyz="-0.25 0 0" rpy="0 0 0"/>
@@ -466,5 +566,11 @@
         <color rgba="0.35 0.37 0.40 1.0"/>
       </material>
-    </visual>
+    </visual></xacro:unless>
+    <xacro:if value="$(arg detailed_visuals)">
+      <visual><geometry><mesh filename="package://raptor_description/meshes/raptor/tail_link__graphite.dae"/></geometry><material name="raptor_graphite"><color rgba="0.065 0.075 0.085 1"/></material></visual>
+      <visual><geometry><mesh filename="package://raptor_description/meshes/raptor/tail_link__titanium.dae"/></geometry><material name="raptor_titanium"><color rgba="0.36 0.4 0.43 1"/></material></visual>
+      <visual><geometry><mesh filename="package://raptor_description/meshes/raptor/tail_link__ivory.dae"/></geometry><material name="raptor_ivory"><color rgba="0.72 0.72 0.65 1"/></material></visual>
+      <visual><geometry><mesh filename="package://raptor_description/meshes/raptor/tail_link__copper.dae"/></geometry><material name="raptor_copper"><color rgba="0.66 0.29 0.08 1"/></material></visual>
+    </xacro:if>
     <collision>
       <origin xyz="-0.25 0 0" rpy="0 0 0"/>

Commit message: feat: add passive articulated toes and measured terrain contact tests

File: src/raptor_description/urdf/raptor.urdf.xacro (robot description, xacro)
@@ -7,4 +7,9 @@
   <xacro:arg name="detailed_visuals" default="false"/>
   <xacro:arg name="sensors" default="false"/>
+  <xacro:arg name="passive_toes" default="false"/>
+  <xacro:arg name="crouched_start" default="false"/>
+  <xacro:arg name="crouch_hip_pitch" default="-0.15"/>
+  <xacro:property name="crouch_hip" value="$(arg crouch_hip_pitch)"/>
+  <xacro:include filename="passive_toes.xacro"/>
   <xacro:if value="$(arg sensors)">
     <gazebo reference="base_link">
@@ -12,4 +17,5 @@
         <always_on>true</always_on><update_rate>50</update_rate>
         <topic>/raptor/imu</topic>
+        <imu><orientation_reference_frame><localization>ENU</localization></orientation_reference_frame></imu>
       </sensor>
       <sensor name="front_rgbd" type="rgbd_camera">
@@ -259,4 +265,5 @@
   <!-- 발목을 앞뒤로 움직이는 네 번째 관절 -->
   <!-- ========================================= -->
+  <xacro:unless value="$(arg passive_toes)">
   <link name="left_foot_link">
     <xacro:unless value="$(arg detailed_visuals)"><visual>
@@ -294,4 +301,6 @@
     </inertial>
   </link>
+  </xacro:unless>
+  <xacro:if value="$(arg passive_toes)"><xacro:passive_foot side="left"/></xacro:if>
   <joint name="left_ankle_pitch_joint" type="revolute">
     <parent link="left_shin_link"/>
@@ -455,4 +464,5 @@
   </joint>
   <!-- 4. RIGHT ANKLE PITCH + FOOT -->
+  <xacro:unless value="$(arg passive_toes)">
   <link name="right_foot_link">
     <xacro:unless value="$(arg detailed_visuals)"><visual>
@@ -489,4 +499,6 @@
     </inertial>
   </link>
+  </xacro:unless>
+  <xacro:if value="$(arg passive_toes)"><xacro:passive_foot side="right"/></xacro:if>
   <joint name="right_ankle_pitch_joint" type="revolute">
     <parent link="right_shin_link"/>
@@ -620,15 +632,15 @@
     <joint name="left_hip_pitch_joint">
       <command_interface name="position"/>
-      <state_interface name="position"/>
+      <state_interface name="position"><xacro:if value="$(arg crouched_start)"><param name="initial_value">${crouch_hip}</param></xacro:if></state_interface>
       <state_interface name="velocity"/>
     </joint>
     <joint name="left_knee_pitch_joint">
       <command_interface name="position"/>
-      <state_interface name="position"/>
+      <state_interface name="position"><xacro:if value="$(arg crouched_start)"><param name="initial_value">0.4</param></xacro:if></state_interface>
       <state_interface name="velocity"/>
     </joint>
     <joint name="left_ankle_pitch_joint">
       <command_interface name="position"/>
-      <state_interface name="position"/>
+      <state_interface name="position"><xacro:if value="$(arg crouched_start)"><param name="initial_value">${-0.4-crouch_hip}</param></xacro:if></state_interface>
       <state_interface name="velocity"/>
     </joint>
@@ -641,15 +653,15 @@
     <joint name="right_hip_pitch_joint">
       <command_interface name="position"/>
-      <state_interface name="position"/>
+      <state_interface name="position"><xacro:if value="$(arg crouched_start)"><param name="initial_value">${crouch_hip}</param></xacro:if></state_interface>
       <state_interface name="velocity"/>
     </joint>
     <joint name="right_knee_pitch_joint">
       <command_interface name="position"/>
-      <state_interface name="position"/>
+      <state_interface name="position"><xacro:if value="$(arg crouched_start)"><param name="initial_value">0.4</param></xacro:if></state_interface>
       <state_interface name="velocity"/>
     </joint>
     <joint name="right_ankle_pitch_joint">
       <command_interface name="position"/>
-      <state_interface name="position"/>
+      <state_interface name="position"><xacro:if value="$(arg crouched_start)"><param name="initial_value">${-0.4-crouch_hip}</param></xacro:if></state_interface>
       <state_interface name="velocity"/>
     </joint>
@@ -680,3 +692,20 @@
     </plugin>
   </gazebo>
+  <xacro:if value="$(arg passive_toes)">
+    <gazebo><plugin filename="gz-sim-joint-state-publisher-system" name="gz::sim::systems::JointStatePublisher">
+      <topic>/raptor/passive_joint_states</topic><update_rate>50</update_rate>
+      <joint_name>left_toe_1_proximal_joint</joint_name>
+      <joint_name>left_toe_1_distal_joint</joint_name>
+      <joint_name>left_toe_2_proximal_joint</joint_name>
+      <joint_name>left_toe_2_distal_joint</joint_name>
+      <joint_name>left_toe_3_proximal_joint</joint_name>
+      <joint_name>left_toe_3_distal_joint</joint_name>
+      <joint_name>right_toe_1_proximal_joint</joint_name>
+      <joint_name>right_toe_1_distal_joint</joint_name>
+      <joint_name>right_toe_2_proximal_joint</joint_name>
+      <joint_name>right_toe_2_distal_joint</joint_name>
+      <joint_name>right_toe_3_proximal_joint</joint_name>
+      <joint_name>right_toe_3_distal_joint</joint_name>
+    </plugin></gazebo>
+  </xacro:if>
 </robot>
