Commit message: refactor(urdf): leg lengths as xacro properties
Generated URDF numerically identical (default and passive_toes+detailed).

Co-Authored-By: Claude Opus 5.5 <noreply@anthropic.com>

File: src/raptor_description/urdf/raptor.urdf.xacro (robot description, xacro)
@@ -13,4 +13,8 @@
   <xacro:arg name="crouch_hip_pitch" default="-0.15"/>
   <xacro:property name="crouch_hip" value="$(arg crouch_hip_pitch)"/>
+  <!-- Leg proportions (m). Link inertias below are still literal values for these lengths. -->
+  <xacro:property name="hip_drop" value="0.12"/>
+  <xacro:property name="thigh_length" value="0.32"/>
+  <xacro:property name="shin_length" value="0.30"/>
   <xacro:include filename="passive_toes.xacro"/>
   <xacro:if value="$(arg sensors)">
@@ -162,7 +166,7 @@
     <xacro:unless value="$(arg detailed_visuals)"><visual>
       <!-- 관절에서 아래쪽으로 허벅지가 내려감 -->
-      <origin xyz="0 0 -0.16" rpy="0 0 0"/>
-      <geometry>
-        <box size="0.10 0.10 0.32"/>
+      <origin xyz="0 0 ${-thigh_length/2}" rpy="0 0 0"/>
+      <geometry>
+        <box size="0.10 0.10 ${thigh_length}"/>
       </geometry>
       <material name="leg_gray">
@@ -177,11 +181,11 @@
     </xacro:if>
     <collision>
-      <origin xyz="0 0 -0.16" rpy="0 0 0"/>
-      <geometry>
-        <box size="0.10 0.10 0.32"/>
-      </geometry>
-    </collision>
-    <inertial>
-      <origin xyz="0 0 -0.16" rpy="0 0 0"/>
+      <origin xyz="0 0 ${-thigh_length/2}" rpy="0 0 0"/>
+      <geometry>
+        <box size="0.10 0.10 ${thigh_length}"/>
+      </geometry>
+    </collision>
+    <inertial>
+      <origin xyz="0 0 ${-thigh_length/2}" rpy="0 0 0"/>
       <mass value="1.5"/>
       <inertia
@@ -198,5 +202,5 @@
     <child link="left_thigh_link"/>
     <!-- Hip Roll 블록 아래쪽에 Hip Pitch 배치 -->
-    <origin xyz="0 0 -0.12" rpy="0 0 0"/>
+    <origin xyz="0 0 ${-hip_drop}" rpy="0 0 0"/>
     <!-- Y축 회전 = 다리 앞뒤 움직임 -->
     <axis xyz="0 1 0"/>
@@ -215,7 +219,7 @@
     <xacro:unless value="$(arg detailed_visuals)"><visual>
       <!-- 무릎 아래로 종아리가 내려감 -->
-      <origin xyz="0 0 -0.15" rpy="0 0 0"/>
-      <geometry>
-        <box size="0.085 0.085 0.30"/>
+      <origin xyz="0 0 ${-shin_length/2}" rpy="0 0 0"/>
+      <geometry>
+        <box size="0.085 0.085 ${shin_length}"/>
       </geometry>
       <material name="shin_gray">
@@ -229,11 +233,11 @@
     </xacro:if>
     <collision>
-      <origin xyz="0 0 -0.15" rpy="0 0 0"/>
-      <geometry>
-        <box size="0.085 0.085 0.30"/>
-      </geometry>
-    </collision>
-    <inertial>
-      <origin xyz="0 0 -0.15" rpy="0 0 0"/>
+      <origin xyz="0 0 ${-shin_length/2}" rpy="0 0 0"/>
+      <geometry>
+        <box size="0.085 0.085 ${shin_length}"/>
+      </geometry>
+    </collision>
+    <inertial>
+      <origin xyz="0 0 ${-shin_length/2}" rpy="0 0 0"/>
       <mass value="1.1"/>
       <inertia
@@ -250,5 +254,5 @@
     <child link="left_shin_link"/>
     <!-- 허벅지 끝 = 무릎 위치 -->
-    <origin xyz="0 0 -0.32" rpy="0 0 0"/>
+    <origin xyz="0 0 ${-thigh_length}" rpy="0 0 0"/>
     <!-- Y축 회전 = 무릎 굽힘 -->
     <axis xyz="0 1 0"/>
@@ -309,5 +313,5 @@
     <child link="left_foot_link"/>
     <!-- 종아리 끝부분에 발목 배치 -->
-    <origin xyz="0 0 -0.30" rpy="0 0 0"/>
+    <origin xyz="0 0 ${-shin_length}" rpy="0 0 0"/>
     <!-- Y축 회전 = 발 앞뒤 기울임 -->
     <axis xyz="0 1 0"/>
@@ -376,7 +380,7 @@
   <link name="right_thigh_link">
     <xacro:unless value="$(arg detailed_visuals)"><visual>
-      <origin xyz="0 0 -0.16" rpy="0 0 0"/>
-      <geometry>
-        <box size="0.10 0.10 0.32"/>
+      <origin xyz="0 0 ${-thigh_length/2}" rpy="0 0 0"/>
+      <geometry>
+        <box size="0.10 0.10 ${thigh_length}"/>
       </geometry>
       <material name="right_leg_gray">
@@ -391,11 +395,11 @@
     </xacro:if>
     <collision>
-      <origin xyz="0 0 -0.16" rpy="0 0 0"/>
-      <geometry>
-        <box size="0.10 0.10 0.32"/>
-      </geometry>
-    </collision>
-    <inertial>
-      <origin xyz="0 0 -0.16" rpy="0 0 0"/>
+      <origin xyz="0 0 ${-thigh_length/2}" rpy="0 0 0"/>
+      <geometry>
+        <box size="0.10 0.10 ${thigh_length}"/>
+      </geometry>
+    </collision>
+    <inertial>
+      <origin xyz="0 0 ${-thigh_length/2}" rpy="0 0 0"/>
       <mass value="1.5"/>
       <inertia
@@ -411,5 +415,5 @@
     <parent link="right_hip_roll_link"/>
     <child link="right_thigh_link"/>
-    <origin xyz="0 0 -0.12" rpy="0 0 0"/>
+    <origin xyz="0 0 ${-hip_drop}" rpy="0 0 0"/>
     <!-- 앞 / 뒤 -->
     <axis xyz="0 1 0"/>
@@ -423,7 +427,7 @@
   <link name="right_shin_link">
     <xacro:unless value="$(arg detailed_visuals)"><visual>
-      <origin xyz="0 0 -0.15" rpy="0 0 0"/>
-      <geometry>
-        <box size="0.085 0.085 0.30"/>
+      <origin xyz="0 0 ${-shin_length/2}" rpy="0 0 0"/>
+      <geometry>
+        <box size="0.085 0.085 ${shin_length}"/>
       </geometry>
       <material name="right_shin_gray">
@@ -437,11 +441,11 @@
     </xacro:if>
     <collision>
-      <origin xyz="0 0 -0.15" rpy="0 0 0"/>
-      <geometry>
-        <box size="0.085 0.085 0.30"/>
-      </geometry>
-    </collision>
-    <inertial>
-      <origin xyz="0 0 -0.15" rpy="0 0 0"/>
+      <origin xyz="0 0 ${-shin_length/2}" rpy="0 0 0"/>
+      <geometry>
+        <box size="0.085 0.085 ${shin_length}"/>
+      </geometry>
+    </collision>
+    <inertial>
+      <origin xyz="0 0 ${-shin_length/2}" rpy="0 0 0"/>
       <mass value="1.1"/>
       <inertia
@@ -457,5 +461,5 @@
     <parent link="right_thigh_link"/>
     <child link="right_shin_link"/>
-    <origin xyz="0 0 -0.32" rpy="0 0 0"/>
+    <origin xyz="0 0 ${-thigh_length}" rpy="0 0 0"/>
     <axis xyz="0 1 0"/>
     <limit
@@ -506,5 +510,5 @@
     <parent link="right_shin_link"/>
     <child link="right_foot_link"/>
-    <origin xyz="0 0 -0.30" rpy="0 0 0"/>
+    <origin xyz="0 0 ${-shin_length}" rpy="0 0 0"/>
     <axis xyz="0 1 0"/>
     <limit

Commit message: feat(model): ankle_pitch_limit override (design variant +-1.0 rad); --model for RL
The 12-DOF gait held the ankle at its -0.70 stop 42% of the time; a 0.55 margin broke it.

Co-Authored-By: Claude Opus 5.5 <noreply@anthropic.com>

File: src/raptor_description/urdf/raptor.urdf.xacro (robot description, xacro)
@@ -31,5 +31,8 @@
   <xacro:if value="${ankle_roll and legacy}"><xacro:ERROR_ankle_roll_needs_a_digitigrade_leg_design/></xacro:if>
   <xacro:property name="hip_drop" value="${0.06 if low else 0.12}"/>
-  <xacro:property name="ankle_limit" value="${0.95 if low else 0.70}"/>
+  <!-- ankle_pitch_limit: optional override (rad). The 12-DOF flat-pad RL gait held the ankle at the -0.70 stop
+       42% of the time (evidence 82); the feasibility study recommended a wider range. 0 = design default. -->
+  <xacro:arg name="ankle_pitch_limit" default="0"/>
+  <xacro:property name="ankle_limit" value="${float('$(arg ankle_pitch_limit)') if float('$(arg ankle_pitch_limit)') > 0 else (0.95 if low else 0.70)}"/>
   <xacro:property name="toe_splay" value="${0.35 if low else 0.12}"/>
   <xacro:property name="thigh_length" value="${0.32 if legacy else 0.26}"/>
