Commit message: feat: share articulated toe visuals and track persistent work

File: src/raptor_description/urdf/passive_toes.xacro (robot description, xacro)
@@ -6,4 +6,5 @@
     <xacro:property name="joint_name" value="${side}_toe_${digit}_${part}_joint"/>
     <link name="${link_name}">
+      <xacro:unless value="$(arg detailed_visuals)">
       <visual><origin xyz="${length/2} 0 0"/>
         <geometry><box size="${length} 0.026 0.034"/></geometry>
@@ -20,4 +21,11 @@
           <geometry><box size="0.026 0.012 0.013"/></geometry>
           <material name="toe_claw"><color rgba="0.12 0.14 0.16 1"/></material></visual>
+      </xacro:if>
+      </xacro:unless>
+      <xacro:if value="$(arg detailed_visuals)">
+        <visual><geometry><mesh filename="package://raptor_description/meshes/raptor/toe_${part}__graphite.dae"/></geometry><material name="toe_detail_graphite"><color rgba=".065 .075 .085 1"/></material></visual>
+        <visual><geometry><mesh filename="package://raptor_description/meshes/raptor/toe_${part}__ivory.dae"/></geometry><material name="toe_detail_ivory"><color rgba=".72 .72 .65 1"/></material></visual>
+        <visual><geometry><mesh filename="package://raptor_description/meshes/raptor/toe_${part}__titanium.dae"/></geometry><material name="toe_detail_titanium"><color rgba=".36 .40 .43 1"/></material></visual>
+        <visual><geometry><mesh filename="package://raptor_description/meshes/raptor/toe_${part}__rubber.dae"/></geometry><material name="toe_detail_rubber"><color rgba=".025 .028 .032 1"/></material></visual>
       </xacro:if>
       <collision><origin xyz="${length/2} 0 0"/>
@@ -58,4 +66,5 @@
   <xacro:macro name="passive_foot" params="side">
     <link name="${side}_foot_link">
+      <xacro:unless value="$(arg detailed_visuals)">
       <visual><origin xyz="-0.015 0 -0.03"/>
         <geometry><box size="0.09 0.10 0.06"/></geometry>
@@ -64,4 +73,11 @@
         <geometry><cylinder radius="0.037" length="0.10"/></geometry>
         <material name="ankle_housing"><color rgba="0.36 0.40 0.43 1"/></material></visual>
+      </xacro:unless>
+      <xacro:if value="$(arg detailed_visuals)">
+        <visual><geometry><mesh filename="package://raptor_description/meshes/raptor/passive_heel__graphite.dae"/></geometry><material name="heel_detail_graphite"><color rgba=".065 .075 .085 1"/></material></visual>
+        <visual><geometry><mesh filename="package://raptor_description/meshes/raptor/passive_heel__ivory.dae"/></geometry><material name="heel_detail_ivory"><color rgba=".72 .72 .65 1"/></material></visual>
+        <visual><geometry><mesh filename="package://raptor_description/meshes/raptor/passive_heel__titanium.dae"/></geometry><material name="heel_detail_titanium"><color rgba=".36 .40 .43 1"/></material></visual>
+        <visual><geometry><mesh filename="package://raptor_description/meshes/raptor/passive_heel__rubber.dae"/></geometry><material name="heel_detail_rubber"><color rgba=".025 .028 .032 1"/></material></visual>
+      </xacro:if>
       <collision><origin xyz="-0.015 0 -0.03"/>
         <geometry><box size="0.09 0.10 0.06"/></geometry></collision>

Commit message: test: isolate passive toe stiffness effect on support transition

File: src/raptor_description/urdf/passive_toes.xacro (robot description, xacro)
@@ -43,5 +43,5 @@
     </joint>
     <gazebo reference="${joint_name}">
-      <springReference>0</springReference><springStiffness>${stiffness}</springStiffness>
+      <springReference>0</springReference><springStiffness>${stiffness * toe_stiffness_scale}</springStiffness>
     </gazebo>
     <gazebo reference="${link_name}">

File: src/raptor_description/urdf/raptor.urdf.xacro (robot description, xacro)
@@ -8,4 +8,6 @@
   <xacro:arg name="sensors" default="false"/>
   <xacro:arg name="passive_toes" default="false"/>
+  <xacro:arg name="toe_stiffness_scale" default="1.0"/>
+  <xacro:property name="toe_stiffness_scale" value="$(arg toe_stiffness_scale)"/>
   <xacro:arg name="crouched_start" default="false"/>
   <xacro:arg name="crouch_hip_pitch" default="-0.15"/>
