Commit message: feat(urdf): digitigrade leg design option with 10 active DOF
leg_design:=digitigrade: shorter thigh, inclined metatarsus foot with rigid
pad and passive toes. Legacy URDF numerically unchanged. MuJoCo: better
standing, rocking 9/9, stride without falls at kv100; Gazebo stands.

Co-Authored-By: Claude Opus 5.5 <noreply@anthropic.com>

File: src/raptor_description/urdf/passive_toes.xacro (robot description, xacro)
@@ -56,7 +56,7 @@
     </gazebo>
   </xacro:macro>
-  <xacro:macro name="toe_digit" params="side digit y yaw">
+  <xacro:macro name="toe_digit" params="side digit y yaw x0:=0.005 z0:=-0.043">
     <xacro:toe_segment side="${side}" digit="${digit}" part="proximal"
-      parent="${side}_foot_link" xyz="0.005 ${y} -0.043" yaw="${yaw}"
+      parent="${side}_foot_link" xyz="${x0} ${y} ${z0}" yaw="${yaw}"
       length="0.070" stiffness="12"/>
     <xacro:toe_segment side="${side}" digit="${digit}" part="distal"

File: src/raptor_description/urdf/raptor.urdf.xacro (robot description, xacro)
@@ -14,8 +14,21 @@
   <xacro:property name="crouch_hip" value="$(arg crouch_hip_pitch)"/>
   <!-- Leg proportions (m). Link inertias below are still literal values for these lengths. -->
+  <!-- legacy: original straight leg and flat foot (reproduces evidence 01-62).
+       digitigrade: shorter thigh + inclined metatarsus foot, still 10 active DOF. -->
+  <xacro:arg name="leg_design" default="legacy"/>
+  <!-- Unknown values fail with a KeyError instead of silently picking a design. -->
+  <xacro:property name="legacy" value="${dict(legacy=True, digitigrade=False)['$(arg leg_design)']}"/>
   <xacro:property name="hip_drop" value="0.12"/>
-  <xacro:property name="thigh_length" value="0.32"/>
+  <xacro:property name="thigh_length" value="${0.32 if legacy else 0.26}"/>
   <xacro:property name="shin_length" value="0.30"/>
+  <!-- Legacy inertias are the original literals; digitigrade uses the box formula. -->
+  <xacro:property name="thigh_ixx" value="${0.0140 if legacy else 1.5*(0.10**2+thigh_length**2)/12}"/>
+  <xacro:property name="shin_ixx" value="${0.0089 if legacy else 1.1*(0.085**2+shin_length**2)/12}"/>
+  <!-- Legacy thigh/shin meshes fit only the legacy lengths. -->
+  <xacro:property name="leg_meshes" value="${'$(arg detailed_visuals)' == 'true' and legacy}"/>
   <xacro:include filename="passive_toes.xacro"/>
+  <xacro:include filename="digitigrade_foot.xacro"/>
+  <!-- crouched_start knee; the ankle keeps the sole level (hip + knee + ankle = 0). -->
+  <xacro:property name="crouch_knee" value="${0.4 if legacy else 0.5}"/>
   <xacro:if value="$(arg sensors)">
     <gazebo reference="base_link">
@@ -164,5 +177,5 @@
   <!-- ========================================= -->
   <link name="left_thigh_link">
-    <xacro:unless value="$(arg detailed_visuals)"><visual>
+    <xacro:unless value="${leg_meshes}"><visual>
       <!-- 관절에서 아래쪽으로 허벅지가 내려감 -->
       <origin xyz="0 0 ${-thigh_length/2}" rpy="0 0 0"/>
@@ -174,5 +187,5 @@
       </material>
     </visual></xacro:unless>
-    <xacro:if value="$(arg detailed_visuals)">
+    <xacro:if value="${leg_meshes}">
       <visual><geometry><mesh filename="package://raptor_description/meshes/raptor/left_thigh_link__graphite.dae"/></geometry><material name="raptor_graphite"><color rgba="0.065 0.075 0.085 1"/></material></visual>
       <visual><geometry><mesh filename="package://raptor_description/meshes/raptor/left_thigh_link__titanium.dae"/></geometry><material name="raptor_titanium"><color rgba="0.36 0.4 0.43 1"/></material></visual>
@@ -190,8 +203,8 @@
       <mass value="1.5"/>
       <inertia
-        ixx="0.0140"
-        ixy="0.0"
-        ixz="0.0"
-        iyy="0.0140"
+        ixx="${thigh_ixx}"
+        ixy="0.0"
+        ixz="0.0"
+        iyy="${thigh_ixx}"
         iyz="0.0"
         izz="0.0025"/>
@@ -217,5 +230,5 @@
   <!-- ========================================= -->
   <link name="left_shin_link">
-    <xacro:unless value="$(arg detailed_visuals)"><visual>
+    <xacro:unless value="${leg_meshes}"><visual>
       <!-- 무릎 아래로 종아리가 내려감 -->
       <origin xyz="0 0 ${-shin_length/2}" rpy="0 0 0"/>
@@ -227,5 +240,5 @@
       </material>
     </visual></xacro:unless>
-    <xacro:if value="$(arg detailed_visuals)">
+    <xacro:if value="${leg_meshes}">
       <visual><geometry><mesh filename="package://raptor_description/meshes/raptor/left_shin_link__graphite.dae"/></geometry><material name="raptor_graphite"><color rgba="0.065 0.075 0.085 1"/></material></visual>
       <visual><geometry><mesh filename="package://raptor_description/meshes/raptor/left_shin_link__titanium.dae"/></geometry><material name="raptor_titanium"><color rgba="0.36 0.4 0.43 1"/></material></visual>
@@ -242,8 +255,8 @@
       <mass value="1.1"/>
       <inertia
-        ixx="0.0089"
-        ixy="0.0"
-        ixz="0.0"
-        iyy="0.0089"
+        ixx="${shin_ixx}"
+        ixy="0.0"
+        ixz="0.0"
+        iyy="${shin_ixx}"
         iyz="0.0"
         izz="0.0013"/>
@@ -271,4 +284,5 @@
   <!-- 발목을 앞뒤로 움직이는 네 번째 관절 -->
   <!-- ========================================= -->
+  <xacro:if value="${legacy}">
   <xacro:unless value="$(arg passive_toes)">
   <link name="left_foot_link">
@@ -309,4 +323,6 @@
   </xacro:unless>
   <xacro:if value="$(arg passive_toes)"><xacro:passive_foot side="left"/></xacro:if>
+  </xacro:if>
+  <xacro:unless value="${legacy}"><xacro:digitigrade_foot side="left" passive="$(arg passive_toes)"/></xacro:unless>
   <joint name="left_ankle_pitch_joint" type="revolute">
     <parent link="left_shin_link"/>
@@ -379,5 +395,5 @@
   <!-- 2. RIGHT HIP PITCH + THIGH -->
   <link name="right_thigh_link">
-    <xacro:unless value="$(arg detailed_visuals)"><visual>
+    <xacro:unless value="${leg_meshes}"><visual>
       <origin xyz="0 0 ${-thigh_length/2}" rpy="0 0 0"/>
       <geometry>
@@ -388,5 +404,5 @@
       </material>
     </visual></xacro:unless>
-    <xacro:if value="$(arg detailed_visuals)">
+    <xacro:if value="${leg_meshes}">
       <visual><geometry><mesh filename="package://raptor_description/meshes/raptor/right_thigh_link__graphite.dae"/></geometry><material name="raptor_graphite"><color rgba="0.065 0.075 0.085 1"/></material></visual>
       <visual><geometry><mesh filename="package://raptor_description/meshes/raptor/right_thigh_link__titanium.dae"/></geometry><material name="raptor_titanium"><color rgba="0.36 0.4 0.43 1"/></material></visual>
@@ -404,8 +420,8 @@
       <mass value="1.5"/>
       <inertia
-        ixx="0.0140"
-        ixy="0.0"
-        ixz="0.0"
-        iyy="0.0140"
+        ixx="${thigh_ixx}"
+        ixy="0.0"
+        ixz="0.0"
+        iyy="${thigh_ixx}"
         iyz="0.0"
         izz="0.0025"/>
@@ -426,5 +442,5 @@
   <!-- 3. RIGHT KNEE PITCH + SHIN -->
   <link name="right_shin_link">
-    <xacro:unless value="$(arg detailed_visuals)"><visual>
+    <xacro:unless value="${leg_meshes}"><visual>
       <origin xyz="0 0 ${-shin_length/2}" rpy="0 0 0"/>
       <geometry>
@@ -435,5 +451,5 @@
       </material>
     </visual></xacro:unless>
-    <xacro:if value="$(arg detailed_visuals)">
+    <xacro:if value="${leg_meshes}">
       <visual><geometry><mesh filename="package://raptor_description/meshes/raptor/right_shin_link__graphite.dae"/></geometry><material name="raptor_graphite"><color rgba="0.065 0.075 0.085 1"/></material></visual>
       <visual><geometry><mesh filename="package://raptor_description/meshes/raptor/right_shin_link__titanium.dae"/></geometry><material name="raptor_titanium"><color rgba="0.36 0.4 0.43 1"/></material></visual>
@@ -450,8 +466,8 @@
       <mass value="1.1"/>
       <inertia
-        ixx="0.0089"
-        ixy="0.0"
-        ixz="0.0"
-        iyy="0.0089"
+        ixx="${shin_ixx}"
+        ixy="0.0"
+        ixz="0.0"
+        iyy="${shin_ixx}"
         iyz="0.0"
         izz="0.0013"/>
@@ -470,4 +486,5 @@
   </joint>
   <!-- 4. RIGHT ANKLE PITCH + FOOT -->
+  <xacro:if value="${legacy}">
   <xacro:unless value="$(arg passive_toes)">
   <link name="right_foot_link">
@@ -507,4 +524,6 @@
   </xacro:unless>
   <xacro:if value="$(arg passive_toes)"><xacro:passive_foot side="right"/></xacro:if>
+  </xacro:if>
+  <xacro:unless value="${legacy}"><xacro:digitigrade_foot side="right" passive="$(arg passive_toes)"/></xacro:unless>
   <joint name="right_ankle_pitch_joint" type="revolute">
     <parent link="right_shin_link"/>
@@ -645,5 +664,5 @@
     <joint name="left_knee_pitch_joint">
       <command_interface name="position"/>
-      <state_interface name="position"><xacro:if value="$(arg crouched_start)"><param name="initial_value">0.4</param></xacro:if></state_interface>
+      <state_interface name="position"><xacro:if value="$(arg crouched_start)"><param name="initial_value">${crouch_knee}</param></xacro:if></state_interface>
       <state_interface name="velocity"/>
       <state_interface name="effort"/>
@@ -651,5 +670,5 @@
     <joint name="left_ankle_pitch_joint">
       <command_interface name="position"/>
-      <state_interface name="position"><xacro:if value="$(arg crouched_start)"><param name="initial_value">${-0.4-crouch_hip}</param></xacro:if></state_interface>
+      <state_interface name="position"><xacro:if value="$(arg crouched_start)"><param name="initial_value">${-crouch_knee-crouch_hip}</param></xacro:if></state_interface>
       <state_interface name="velocity"/>
       <state_interface name="effort"/>
@@ -670,5 +689,5 @@
     <joint name="right_knee_pitch_joint">
       <command_interface name="position"/>
-      <state_interface name="position"><xacro:if value="$(arg crouched_start)"><param name="initial_value">0.4</param></xacro:if></state_interface>
+      <state_interface name="position"><xacro:if value="$(arg crouched_start)"><param name="initial_value">${crouch_knee}</param></xacro:if></state_interface>
       <state_interface name="velocity"/>
       <state_interface name="effort"/>
@@ -676,5 +695,5 @@
     <joint name="right_ankle_pitch_joint">
       <command_interface name="position"/>
-      <state_interface name="position"><xacro:if value="$(arg crouched_start)"><param name="initial_value">${-0.4-crouch_hip}</param></xacro:if></state_interface>
+      <state_interface name="position"><xacro:if value="$(arg crouched_start)"><param name="initial_value">${-crouch_knee-crouch_hip}</param></xacro:if></state_interface>
       <state_interface name="velocity"/>
       <state_interface name="effort"/>
