Commit message: feat(urdf): digitigrade Morphloom GLB visuals
Used only for leg_design:=digitigrade with detailed_visuals; legacy URDF
numerically unchanged. glTF Y-up corrected with a visual origin roll.

Co-Authored-By: Claude Opus 5.5 <noreply@anthropic.com>

File: src/raptor_description/urdf/digitigrade_foot.xacro (robot description, xacro)
@@ -23,4 +23,6 @@
     <xacro:property name="foot_mass" value="${0.3 if passive else 0.6}"/>
     <link name="${side}_foot_link">
+      <xacro:dg_visual link="${side}_foot_link"/>
+      <xacro:unless value="${detailed}">
       <visual><origin xyz="${pad_x} 0 ${pad_z}"/>
         <geometry><box size="${pad_length} ${pad_width} ${pad_thickness}"/></geometry>
@@ -29,4 +31,5 @@
         <geometry><box size="${meta_width} ${meta_width} ${meta_length}"/></geometry>
         <material name="metatarsus_gray"><color rgba="0.42 0.44 0.47 1"/></material></visual>
+      </xacro:unless>
       <collision><origin xyz="${pad_x} 0 ${pad_z}"/>
         <geometry><box size="${pad_length} ${pad_width} ${pad_thickness}"/></geometry></collision>

File: src/raptor_description/urdf/passive_toes.xacro (robot description, xacro)
@@ -6,5 +6,6 @@
     <xacro:property name="joint_name" value="${side}_toe_${digit}_${part}_joint"/>
     <link name="${link_name}">
-      <xacro:unless value="$(arg detailed_visuals)">
+      <xacro:dg_visual link="${link_name}"/>
+      <xacro:unless value="${detailed}">
       <visual><origin xyz="${length/2} 0 0"/>
         <geometry><box size="${length} 0.026 0.034"/></geometry>
@@ -23,5 +24,5 @@
       </xacro:if>
       </xacro:unless>
-      <xacro:if value="$(arg detailed_visuals)">
+      <xacro:if value="${legacy_detail}">
         <visual><geometry><mesh filename="package://raptor_description/meshes/raptor/toe_${part}__graphite.dae"/></geometry><material name="toe_detail_graphite"><color rgba=".065 .075 .085 1"/></material></visual>
         <visual><geometry><mesh filename="package://raptor_description/meshes/raptor/toe_${part}__ivory.dae"/></geometry><material name="toe_detail_ivory"><color rgba=".72 .72 .65 1"/></material></visual>
@@ -66,5 +67,5 @@
   <xacro:macro name="passive_foot" params="side">
     <link name="${side}_foot_link">
-      <xacro:unless value="$(arg detailed_visuals)">
+      <xacro:unless value="${detailed}">
       <visual><origin xyz="-0.015 0 -0.03"/>
         <geometry><box size="0.09 0.10 0.06"/></geometry>
@@ -74,5 +75,5 @@
         <material name="ankle_housing"><color rgba="0.36 0.40 0.43 1"/></material></visual>
       </xacro:unless>
-      <xacro:if value="$(arg detailed_visuals)">
+      <xacro:if value="${legacy_detail}">
         <visual><geometry><mesh filename="package://raptor_description/meshes/raptor/passive_heel__graphite.dae"/></geometry><material name="heel_detail_graphite"><color rgba=".065 .075 .085 1"/></material></visual>
         <visual><geometry><mesh filename="package://raptor_description/meshes/raptor/passive_heel__ivory.dae"/></geometry><material name="heel_detail_ivory"><color rgba=".72 .72 .65 1"/></material></visual>

File: src/raptor_description/urdf/raptor.urdf.xacro (robot description, xacro)
@@ -26,5 +26,11 @@
   <xacro:property name="shin_ixx" value="${0.0089 if legacy else 1.1*(0.085**2+shin_length**2)/12}"/>
   <!-- Legacy thigh/shin meshes fit only the legacy lengths. -->
-  <xacro:property name="leg_meshes" value="${'$(arg detailed_visuals)' == 'true' and legacy}"/>
+  <xacro:property name="detailed" value="${'$(arg detailed_visuals)' == 'true'}"/>
+  <!-- legacy_detail: original DAE visuals. dg_detail: per-link Morphloom GLBs (modeling/morphloom). -->
+  <xacro:property name="legacy_detail" value="${detailed and legacy}"/>
+  <xacro:property name="dg_detail" value="${detailed and not legacy}"/>
+  <xacro:macro name="dg_visual" params="link">
+    <xacro:if value="${dg_detail}"><visual><origin rpy="${pi/2} 0 0"/><geometry><mesh filename="package://raptor_description/meshes/digitigrade/${link}.glb"/></geometry></visual></xacro:if>
+  </xacro:macro>
   <xacro:include filename="passive_toes.xacro"/>
   <xacro:include filename="digitigrade_foot.xacro"/>
@@ -83,6 +89,7 @@
   -->
   <link name="base_link">
+    <xacro:dg_visual link="base_link"/>
     <!-- 화면에 보이는 외형 -->
-    <xacro:unless value="$(arg detailed_visuals)"><visual>
+    <xacro:unless value="${detailed}"><visual>
       <origin xyz="0 0 0" rpy="0 0 0"/>
       <geometry>
@@ -93,5 +100,5 @@
       </material>
     </visual></xacro:unless>
-    <xacro:if value="$(arg detailed_visuals)">
+    <xacro:if value="${legacy_detail}">
       <visual><geometry><mesh filename="package://raptor_description/meshes/raptor/base_link__graphite.dae"/></geometry><material name="raptor_graphite"><color rgba="0.065 0.075 0.085 1"/></material></visual>
       <visual><geometry><mesh filename="package://raptor_description/meshes/raptor/base_link__titanium.dae"/></geometry><material name="raptor_titanium"><color rgba="0.36 0.4 0.43 1"/></material></visual>
@@ -126,5 +133,6 @@
     <!-- ========================================= -->
     <link name="left_hip_roll_link">
-    <xacro:unless value="$(arg detailed_visuals)"><visual>
+    <xacro:dg_visual link="left_hip_roll_link"/>
+    <xacro:unless value="${detailed}"><visual>
       <origin xyz="0 0 -0.06" rpy="0 0 0"/>
       <geometry>
@@ -135,5 +143,5 @@
       </material>
     </visual></xacro:unless>
-    <xacro:if value="$(arg detailed_visuals)">
+    <xacro:if value="${legacy_detail}">
       <visual><geometry><mesh filename="package://raptor_description/meshes/raptor/left_hip_roll_link__graphite.dae"/></geometry><material name="raptor_graphite"><color rgba="0.065 0.075 0.085 1"/></material></visual>
       <visual><geometry><mesh filename="package://raptor_description/meshes/raptor/left_hip_roll_link__titanium.dae"/></geometry><material name="raptor_titanium"><color rgba="0.36 0.4 0.43 1"/></material></visual>
@@ -177,5 +185,6 @@
   <!-- ========================================= -->
   <link name="left_thigh_link">
-    <xacro:unless value="${leg_meshes}"><visual>
+    <xacro:dg_visual link="left_thigh_link"/>
+    <xacro:unless value="${detailed}"><visual>
       <!-- 관절에서 아래쪽으로 허벅지가 내려감 -->
       <origin xyz="0 0 ${-thigh_length/2}" rpy="0 0 0"/>
@@ -187,5 +196,5 @@
       </material>
     </visual></xacro:unless>
-    <xacro:if value="${leg_meshes}">
+    <xacro:if value="${legacy_detail}">
       <visual><geometry><mesh filename="package://raptor_description/meshes/raptor/left_thigh_link__graphite.dae"/></geometry><material name="raptor_graphite"><color rgba="0.065 0.075 0.085 1"/></material></visual>
       <visual><geometry><mesh filename="package://raptor_description/meshes/raptor/left_thigh_link__titanium.dae"/></geometry><material name="raptor_titanium"><color rgba="0.36 0.4 0.43 1"/></material></visual>
@@ -230,5 +239,6 @@
   <!-- ========================================= -->
   <link name="left_shin_link">
-    <xacro:unless value="${leg_meshes}"><visual>
+    <xacro:dg_visual link="left_shin_link"/>
+    <xacro:unless value="${detailed}"><visual>
       <!-- 무릎 아래로 종아리가 내려감 -->
       <origin xyz="0 0 ${-shin_length/2}" rpy="0 0 0"/>
@@ -240,5 +250,5 @@
       </material>
     </visual></xacro:unless>
-    <xacro:if value="${leg_meshes}">
+    <xacro:if value="${legacy_detail}">
       <visual><geometry><mesh filename="package://raptor_description/meshes/raptor/left_shin_link__graphite.dae"/></geometry><material name="raptor_graphite"><color rgba="0.065 0.075 0.085 1"/></material></visual>
       <visual><geometry><mesh filename="package://raptor_description/meshes/raptor/left_shin_link__titanium.dae"/></geometry><material name="raptor_titanium"><color rgba="0.36 0.4 0.43 1"/></material></visual>
@@ -287,5 +297,5 @@
   <xacro:unless value="$(arg passive_toes)">
   <link name="left_foot_link">
-    <xacro:unless value="$(arg detailed_visuals)"><visual>
+    <xacro:unless value="${detailed}"><visual>
       <!-- 발목 기준으로 발을 약간 앞으로 배치 -->
       <origin xyz="0.06 0 -0.03" rpy="0 0 0"/>
@@ -297,5 +307,5 @@
       </material>
     </visual></xacro:unless>
-    <xacro:if value="$(arg detailed_visuals)">
+    <xacro:if value="${legacy_detail}">
       <visual><geometry><mesh filename="package://raptor_description/meshes/raptor/left_foot_link__graphite.dae"/></geometry><material name="raptor_graphite"><color rgba="0.065 0.075 0.085 1"/></material></visual>
       <visual><geometry><mesh filename="package://raptor_description/meshes/raptor/left_foot_link__titanium.dae"/></geometry><material name="raptor_titanium"><color rgba="0.36 0.4 0.43 1"/></material></visual>
@@ -345,5 +355,6 @@
   <!-- 1. RIGHT HIP ROLL LINK -->
   <link name="right_hip_roll_link">
-    <xacro:unless value="$(arg detailed_visuals)"><visual>
+    <xacro:dg_visual link="right_hip_roll_link"/>
+    <xacro:unless value="${detailed}"><visual>
       <origin xyz="0 0 -0.06" rpy="0 0 0"/>
       <geometry>
@@ -354,5 +365,5 @@
       </material>
     </visual></xacro:unless>
-    <xacro:if value="$(arg detailed_visuals)">
+    <xacro:if value="${legacy_detail}">
       <visual><geometry><mesh filename="package://raptor_description/meshes/raptor/right_hip_roll_link__graphite.dae"/></geometry><material name="raptor_graphite"><color rgba="0.065 0.075 0.085 1"/></material></visual>
       <visual><geometry><mesh filename="package://raptor_description/meshes/raptor/right_hip_roll_link__titanium.dae"/></geometry><material name="raptor_titanium"><color rgba="0.36 0.4 0.43 1"/></material></visual>
@@ -395,5 +406,6 @@
   <!-- 2. RIGHT HIP PITCH + THIGH -->
   <link name="right_thigh_link">
-    <xacro:unless value="${leg_meshes}"><visual>
+    <xacro:dg_visual link="right_thigh_link"/>
+    <xacro:unless value="${detailed}"><visual>
       <origin xyz="0 0 ${-thigh_length/2}" rpy="0 0 0"/>
       <geometry>
@@ -404,5 +416,5 @@
       </material>
     </visual></xacro:unless>
-    <xacro:if value="${leg_meshes}">
+    <xacro:if value="${legacy_detail}">
       <visual><geometry><mesh filename="package://raptor_description/meshes/raptor/right_thigh_link__graphite.dae"/></geometry><material name="raptor_graphite"><color rgba="0.065 0.075 0.085 1"/></material></visual>
       <visual><geometry><mesh filename="package://raptor_description/meshes/raptor/right_thigh_link__titanium.dae"/></geometry><material name="raptor_titanium"><color rgba="0.36 0.4 0.43 1"/></material></visual>
@@ -442,5 +454,6 @@
   <!-- 3. RIGHT KNEE PITCH + SHIN -->
   <link name="right_shin_link">
-    <xacro:unless value="${leg_meshes}"><visual>
+    <xacro:dg_visual link="right_shin_link"/>
+    <xacro:unless value="${detailed}"><visual>
       <origin xyz="0 0 ${-shin_length/2}" rpy="0 0 0"/>
       <geometry>
@@ -451,5 +464,5 @@
       </material>
     </visual></xacro:unless>
-    <xacro:if value="${leg_meshes}">
+    <xacro:if value="${legacy_detail}">
       <visual><geometry><mesh filename="package://raptor_description/meshes/raptor/right_shin_link__graphite.dae"/></geometry><material name="raptor_graphite"><color rgba="0.065 0.075 0.085 1"/></material></visual>
       <visual><geometry><mesh filename="package://raptor_description/meshes/raptor/right_shin_link__titanium.dae"/></geometry><material name="raptor_titanium"><color rgba="0.36 0.4 0.43 1"/></material></visual>
@@ -489,5 +502,5 @@
   <xacro:unless value="$(arg passive_toes)">
   <link name="right_foot_link">
-    <xacro:unless value="$(arg detailed_visuals)"><visual>
+    <xacro:unless value="${detailed}"><visual>
       <origin xyz="0.06 0 -0.03" rpy="0 0 0"/>
       <geometry>
@@ -498,5 +511,5 @@
       </material>
     </visual></xacro:unless>
-    <xacro:if value="$(arg detailed_visuals)">
+    <xacro:if value="${legacy_detail}">
       <visual><geometry><mesh filename="package://raptor_description/meshes/raptor/right_foot_link__graphite.dae"/></geometry><material name="raptor_graphite"><color rgba="0.065 0.075 0.085 1"/></material></visual>
       <visual><geometry><mesh filename="package://raptor_description/meshes/raptor/right_foot_link__titanium.dae"/></geometry><material name="raptor_titanium"><color rgba="0.36 0.4 0.43 1"/></material></visual>
@@ -544,5 +557,6 @@
   <!-- 몸통 뒤쪽에서 좌우로 회전하는 꼬리 베이스 -->
   <link name="tail_yaw_link">
-    <xacro:unless value="$(arg detailed_visuals)"><visual>
+    <xacro:dg_visual link="tail_yaw_link"/>
+    <xacro:unless value="${detailed}"><visual>
       <!-- 관절 기준 뒤쪽(-X)으로 꼬리 베이스가 뻗음 -->
       <origin xyz="-0.08 0 0" rpy="0 0 0"/>
@@ -554,5 +568,5 @@
       </material>
     </visual></xacro:unless>
-    <xacro:if value="$(arg detailed_visuals)">
+    <xacro:if value="${legacy_detail}">
       <visual><geometry><mesh filename="package://raptor_description/meshes/raptor/tail_yaw_link__graphite.dae"/></geometry><material name="raptor_graphite"><color rgba="0.065 0.075 0.085 1"/></material></visual>
       <visual><geometry><mesh filename="package://raptor_description/meshes/raptor/tail_yaw_link__titanium.dae"/></geometry><material name="raptor_titanium"><color rgba="0.36 0.4 0.43 1"/></material></visual>
@@ -594,5 +608,6 @@
   <!-- 꼬리를 위아래로 움직이는 관절 -->
   <link name="tail_link">
-    <xacro:unless value="$(arg detailed_visuals)"><visual>
+    <xacro:dg_visual link="tail_link"/>
+    <xacro:unless value="${detailed}"><visual>
       <!-- Pitch 관절에서 뒤쪽으로 0.5m 뻗는 꼬리 -->
       <origin xyz="-0.25 0 0" rpy="0 0 0"/>
@@ -604,5 +619,5 @@
       </material>
     </visual></xacro:unless>
-    <xacro:if value="$(arg detailed_visuals)">
+    <xacro:if value="${legacy_detail}">
       <visual><geometry><mesh filename="package://raptor_description/meshes/raptor/tail_link__graphite.dae"/></geometry><material name="raptor_graphite"><color rgba="0.065 0.075 0.085 1"/></material></visual>
       <visual><geometry><mesh filename="package://raptor_description/meshes/raptor/tail_link__titanium.dae"/></geometry><material name="raptor_titanium"><color rgba="0.36 0.4 0.43 1"/></material></visual>

Commit message: feat: digitigrade_low stance and reference-style visuals
Add leg_design:=digitigrade_low to approach the user's Tripo reference look:
hip_drop 0.06, ankle position limit +-0.95, crouch -0.80/1.65/-0.85, wider
passive toe splay. Active DOF, masses, torque/velocity limits and gains are
unchanged; legacy and digitigrade URDFs stay numerically identical.
raptor_parts.py --style reference gives silver armour, chrome rising tail and
longer talons (concept output byte-identical). MuJoCo: standing and rocking
9/9 pass, stride has no falls but fails the clean-step slip criterion.
Gazebo static standing confirmed (evidence 67).

Co-Authored-By: Claude Opus 5.5 <noreply@anthropic.com>

File: src/raptor_description/urdf/digitigrade_foot.xacro (robot description, xacro)
@@ -42,7 +42,7 @@
     </link>
     <xacro:if value="${passive}">
-      <xacro:toe_digit side="${side}" digit="1" y="0.040" yaw="0.12" x0="${pad_x+pad_length/2-0.005}" z0="${pad_z-pad_thickness/2+0.017}"/>
+      <xacro:toe_digit side="${side}" digit="1" y="0.040" yaw="${toe_splay}" x0="${pad_x+pad_length/2-0.005}" z0="${pad_z-pad_thickness/2+0.017}"/>
       <xacro:toe_digit side="${side}" digit="2" y="0" yaw="0" x0="${pad_x+pad_length/2-0.005}" z0="${pad_z-pad_thickness/2+0.017}"/>
-      <xacro:toe_digit side="${side}" digit="3" y="-0.040" yaw="-0.12" x0="${pad_x+pad_length/2-0.005}" z0="${pad_z-pad_thickness/2+0.017}"/>
+      <xacro:toe_digit side="${side}" digit="3" y="-0.040" yaw="${-toe_splay}" x0="${pad_x+pad_length/2-0.005}" z0="${pad_z-pad_thickness/2+0.017}"/>
     </xacro:if>
   </xacro:macro>

File: src/raptor_description/urdf/raptor.urdf.xacro (robot description, xacro)
@@ -15,9 +15,14 @@
   <!-- Leg proportions (m). Link inertias below are still literal values for these lengths. -->
   <!-- legacy: original straight leg and flat foot (reproduces evidence 01-62).
-       digitigrade: shorter thigh + inclined metatarsus foot, still 10 active DOF. -->
+       digitigrade: shorter thigh + inclined metatarsus foot, still 10 active DOF.
+       digitigrade_low: digitigrade links with a lower stance (reference look): hip_drop 0.06,
+       ankle range +-0.95 (position limit only), crouch knee 1.65, wider passive toe splay. -->
   <xacro:arg name="leg_design" default="legacy"/>
   <!-- Unknown values fail with a KeyError instead of silently picking a design. -->
-  <xacro:property name="legacy" value="${dict(legacy=True, digitigrade=False)['$(arg leg_design)']}"/>
-  <xacro:property name="hip_drop" value="0.12"/>
+  <xacro:property name="legacy" value="${dict(legacy=True, digitigrade=False, digitigrade_low=False)['$(arg leg_design)']}"/>
+  <xacro:property name="low" value="${'$(arg leg_design)' == 'digitigrade_low'}"/>
+  <xacro:property name="hip_drop" value="${0.06 if low else 0.12}"/>
+  <xacro:property name="ankle_limit" value="${0.95 if low else 0.70}"/>
+  <xacro:property name="toe_splay" value="${0.35 if low else 0.12}"/>
   <xacro:property name="thigh_length" value="${0.32 if legacy else 0.26}"/>
   <xacro:property name="shin_length" value="0.30"/>
@@ -36,10 +41,10 @@
   <xacro:property name="dg_detail" value="${detailed and not legacy}"/>
   <xacro:macro name="dg_visual" params="link">
-    <xacro:if value="${dg_detail}"><visual><origin rpy="${pi/2} 0 0"/><geometry><mesh filename="package://raptor_description/meshes/digitigrade/${link}.glb"/></geometry></visual></xacro:if>
+    <xacro:if value="${dg_detail}"><visual><origin rpy="${pi/2} 0 0"/><geometry><mesh filename="package://raptor_description/meshes/${'digitigrade_low' if low else 'digitigrade'}/${link}.glb"/></geometry></visual></xacro:if>
   </xacro:macro>
   <xacro:include filename="passive_toes.xacro"/>
   <xacro:include filename="digitigrade_foot.xacro"/>
   <!-- crouched_start knee; the ankle keeps the sole level (hip + knee + ankle = 0). -->
-  <xacro:property name="crouch_knee" value="${0.4 if legacy else 0.5}"/>
+  <xacro:property name="crouch_knee" value="${0.4 if legacy else (1.65 if low else 0.5)}"/>
   <xacro:if value="$(arg sensors)">
     <gazebo reference="base_link">
@@ -349,6 +354,6 @@
     <!-- 약 -40도 ~ +40도 -->
     <limit
-      lower="-0.70"
-      upper="0.70"
+      lower="${-ankle_limit}"
+      upper="${ankle_limit}"
       effort="80"
       velocity="2.5"/>
@@ -550,6 +555,6 @@
     <axis xyz="0 1 0"/>
     <limit
-      lower="-0.70"
-      upper="0.70"
+      lower="${-ankle_limit}"
+      upper="${ankle_limit}"
       effort="80"
       velocity="2.5"/>
