Commit message: feat(model): optional ankle roll (12 active DOF, user decision)
ankle_roll:=true splits the digitigrade foot at the metatarsus end; roll axis just above the pad.
10-DOF URDF/MJCF unchanged. Gazebo: 12 position interfaces, controllers active, stands.
MuJoCo lateral slope static stand: 10 DOF up to 10 deg, 12 DOF up to 20 deg (evidence 77).
RL env reads active joints from the model (--dof 10|12).

Co-Authored-By: Claude Opus 5.5 <noreply@anthropic.com>

File: src/raptor_description/urdf/digitigrade_foot.xacro (robot description, xacro)
@@ -2,5 +2,5 @@
 <robot xmlns:xacro="http://www.ros.org/wiki/xacro">
   <!-- Digitigrade foot link: the ankle joint sits at the top of a forward-inclined metatarsus
-       that ends in a rigid sole pad. Still one link on the existing ankle joint (10 active DOF).
+       that ends in a rigid sole pad. Without ankle_roll: one link on the ankle pitch joint (10 active DOF); with ankle_roll see below.
        The pad is the FIRST collision so <side>_foot_link_collision (contact sensor) is the pad.
        Experimental simulation geometry, not rated hardware. -->
@@ -22,4 +22,5 @@
     <!-- Mass kept equal to the legacy foot variant (0.3 kg with passive toes, else 0.6 kg). -->
     <xacro:property name="foot_mass" value="${0.3 if passive else 0.6}"/>
+    <xacro:unless value="${ankle_roll}">
     <link name="${side}_foot_link">
       <xacro:dg_visual link="${side}_foot_link"/>
@@ -46,4 +47,50 @@
       <xacro:toe_digit side="${side}" digit="3" y="-0.040" yaw="${-toe_splay}" x0="${pad_x+pad_length/2-0.005}" z0="${pad_z-pad_thickness/2+0.017}"/>
     </xacro:if>
+    </xacro:unless>
+    <!-- ankle_roll: the foot splits at the lower end of the metatarsus. The ankle pitch joint drives
+         <side>_metatarsus_link; <side>_ankle_roll_joint (axis x) sits just above the pad, so the pad
+         and toes roll close to the ground. <side>_foot_link stays the pad (contact sensor unchanged).
+         Masses split half/half; total foot mass and pad/toe world geometry at zero pose are unchanged. -->
+    <xacro:if value="${ankle_roll}">
+    <link name="${side}_metatarsus_link">
+      <xacro:dg_visual link="${side}_foot_link"/>
+      <xacro:unless value="${detailed}">
+      <visual><origin xyz="${meta_end_x/2} 0 ${meta_end_z/2}" rpy="0 ${-meta_angle} 0"/>
+        <geometry><box size="${meta_width} ${meta_width} ${meta_length}"/></geometry>
+        <material name="metatarsus_gray"><color rgba="0.42 0.44 0.47 1"/></material></visual>
+      </xacro:unless>
+      <collision><origin xyz="${meta_end_x/2} 0 ${meta_end_z/2}" rpy="0 ${-meta_angle} 0"/>
+        <geometry><box size="${meta_width} ${meta_width} ${meta_length}"/></geometry></collision>
+      <inertial><origin xyz="${meta_end_x/2} 0 ${meta_end_z/2}"/><mass value="${foot_mass/2}"/>
+        <xacro:box_inertia m="${foot_mass/2}" x="${meta_width}" y="${meta_width}" z="${meta_length}"/>
+      </inertial>
+    </link>
+    <joint name="${side}_ankle_roll_joint" type="revolute">
+      <parent link="${side}_metatarsus_link"/>
+      <child link="${side}_foot_link"/>
+      <origin xyz="${meta_end_x} 0 ${meta_end_z}"/>
+      <axis xyz="1 0 0"/>
+      <limit lower="${-ankle_roll_limit}" upper="${ankle_roll_limit}" effort="60" velocity="2.5"/>
+    </joint>
+    <link name="${side}_foot_link">
+      <xacro:unless value="${detailed}">
+      <visual><origin xyz="${pad_x-meta_end_x} 0 ${pad_z-meta_end_z}"/>
+        <geometry><box size="${pad_length} ${pad_width} ${pad_thickness}"/></geometry>
+        <material name="foot_pad_dark"><color rgba="0.08 0.09 0.10 1"/></material></visual>
+      </xacro:unless>
+      <collision><origin xyz="${pad_x-meta_end_x} 0 ${pad_z-meta_end_z}"/>
+        <geometry><box size="${pad_length} ${pad_width} ${pad_thickness}"/></geometry></collision>
+      <inertial><origin xyz="${pad_x-meta_end_x} 0 ${pad_z-meta_end_z}"/><mass value="${foot_mass/2}"/>
+        <xacro:box_inertia m="${foot_mass/2}" x="${pad_length}" y="${pad_width}" z="${pad_thickness}"/>
+      </inertial>
+    </link>
+    <xacro:if value="${passive}">
+      <xacro:property name="tx" value="${pad_x+pad_length/2-0.005-meta_end_x}"/>
+      <xacro:property name="tz" value="${pad_z-pad_thickness/2+0.017-meta_end_z}"/>
+      <xacro:toe_digit side="${side}" digit="1" y="0.040" yaw="${toe_splay}" x0="${tx}" z0="${tz}"/>
+      <xacro:toe_digit side="${side}" digit="2" y="0" yaw="0" x0="${tx}" z0="${tz}"/>
+      <xacro:toe_digit side="${side}" digit="3" y="-0.040" yaw="${-toe_splay}" x0="${tx}" z0="${tz}"/>
+    </xacro:if>
+    </xacro:if>
   </xacro:macro>
 </robot>

File: src/raptor_description/urdf/raptor.urdf.xacro (robot description, xacro)
@@ -22,4 +22,10 @@
   <xacro:property name="legacy" value="${dict(legacy=True, digitigrade=False, digitigrade_low=False)['$(arg leg_design)']}"/>
   <xacro:property name="low" value="${'$(arg leg_design)' == 'digitigrade_low'}"/>
+  <!-- ankle_roll (digitigrade designs only): adds left/right ankle roll, 12 active DOF (user decision
+       2026-09-29). Off by default so the 10-DOF evidence stays reproducible. -->
+  <xacro:arg name="ankle_roll" default="false"/>
+  <xacro:property name="ankle_roll" value="${'$(arg ankle_roll)' == 'true'}"/>
+  <xacro:property name="ankle_roll_limit" value="0.50"/>
+  <xacro:if value="${ankle_roll and legacy}"><xacro:ERROR_ankle_roll_needs_a_digitigrade_leg_design/></xacro:if>
   <xacro:property name="hip_drop" value="${0.06 if low else 0.12}"/>
   <xacro:property name="ankle_limit" value="${0.95 if low else 0.70}"/>
@@ -347,5 +353,5 @@
   <joint name="left_ankle_pitch_joint" type="revolute">
     <parent link="left_shin_link"/>
-    <child link="left_foot_link"/>
+    <child link="${'left_metatarsus_link' if ankle_roll else 'left_foot_link'}"/>
     <!-- 종아리 끝부분에 발목 배치 -->
     <origin xyz="0 0 ${-shin_length}" rpy="0 0 0"/>
@@ -551,5 +557,5 @@
   <joint name="right_ankle_pitch_joint" type="revolute">
     <parent link="right_shin_link"/>
-    <child link="right_foot_link"/>
+    <child link="${'right_metatarsus_link' if ankle_roll else 'right_foot_link'}"/>
     <origin xyz="0 0 ${-shin_length}" rpy="0 0 0"/>
     <axis xyz="0 1 0"/>
@@ -699,4 +705,12 @@
       <state_interface name="effort"/>
     </joint>
+    <xacro:if value="${ankle_roll}">
+    <joint name="left_ankle_roll_joint">
+      <command_interface name="position"/>
+      <state_interface name="position"/>
+      <state_interface name="velocity"/>
+      <state_interface name="effort"/>
+    </joint>
+    </xacro:if>
     <!-- RIGHT LEG -->
     <joint name="right_hip_roll_joint">
@@ -724,4 +738,12 @@
       <state_interface name="effort"/>
     </joint>
+    <xacro:if value="${ankle_roll}">
+    <joint name="right_ankle_roll_joint">
+      <command_interface name="position"/>
+      <state_interface name="position"/>
+      <state_interface name="velocity"/>
+      <state_interface name="effort"/>
+    </joint>
+    </xacro:if>
     <!-- TAIL -->
     <joint name="tail_yaw_joint">
@@ -744,5 +766,5 @@
       name="gz_ros2_control::GazeboSimROS2ControlPlugin">
       <parameters>
-        $(find raptor_control)/config/controllers.yaml
+        $(find raptor_control)/config/${'controllers_ankle_roll.yaml' if ankle_roll else 'controllers.yaml'}
       </parameters>
       <!-- controller가 아직 안 잡은 관절도 현재 위치 유지 -->

Commit message: feat(model): sole_shape:=rocker convex foot pad (option; flat stays default)
Paraboloid-bottom pad mesh (Rx 0.30, Ry 0.20 m), same footprint and mass; binary STL for MuJoCo
and Gazebo. Unassisted stand: flat 10 s+, rocker falls in 1.4 s (needs active balance); adoption
to be decided by matched RL comparison. MJCF mesh paths are relative.

Co-Authored-By: Claude Opus 5.5 <noreply@anthropic.com>

File: src/raptor_description/urdf/digitigrade_foot.xacro (robot description, xacro)
@@ -19,4 +19,9 @@
     <inertia ixx="${m*(y*y+z*z)/12}" ixy="0" ixz="0" iyy="${m*(x*x+z*z)/12}" iyz="0" izz="${m*(x*x+y*y)/12}"/>
   </xacro:macro>
+  <!-- sole_shape: flat (box pad, default) or rocker (convex paraboloid bottom, modeling/build_rocker_pad.py). -->
+  <xacro:macro name="pad_geometry">
+    <xacro:if value="${sole_shape == 'rocker'}"><geometry><mesh filename="package://raptor_description/meshes/foot/rocker_pad.stl"/></geometry></xacro:if>
+    <xacro:unless value="${sole_shape == 'rocker'}"><geometry><box size="${pad_length} ${pad_width} ${pad_thickness}"/></geometry></xacro:unless>
+  </xacro:macro>
   <xacro:macro name="digitigrade_foot" params="side passive">
     <!-- Mass kept equal to the legacy foot variant (0.3 kg with passive toes, else 0.6 kg). -->
@@ -34,5 +39,5 @@
       </xacro:unless>
       <collision><origin xyz="${pad_x} 0 ${pad_z}"/>
-        <geometry><box size="${pad_length} ${pad_width} ${pad_thickness}"/></geometry></collision>
+        <xacro:pad_geometry/></collision>
       <collision><origin xyz="${meta_end_x/2} 0 ${meta_end_z/2}" rpy="0 ${-meta_angle} 0"/>
         <geometry><box size="${meta_width} ${meta_width} ${meta_length}"/></geometry></collision>
@@ -80,5 +85,5 @@
       </xacro:unless>
       <collision><origin xyz="${pad_x-meta_end_x} 0 ${pad_z-meta_end_z}"/>
-        <geometry><box size="${pad_length} ${pad_width} ${pad_thickness}"/></geometry></collision>
+        <xacro:pad_geometry/></collision>
       <inertial><origin xyz="${pad_x-meta_end_x} 0 ${pad_z-meta_end_z}"/><mass value="${foot_mass/2}"/>
         <xacro:box_inertia m="${foot_mass/2}" x="${pad_length}" y="${pad_width}" z="${pad_thickness}"/>

File: src/raptor_description/urdf/raptor.urdf.xacro (robot description, xacro)
@@ -27,4 +27,6 @@
   <xacro:property name="ankle_roll" value="${'$(arg ankle_roll)' == 'true'}"/>
   <xacro:property name="ankle_roll_limit" value="0.50"/>
+  <xacro:arg name="sole_shape" default="flat"/>
+  <xacro:property name="sole_shape" value="${dict(flat='flat', rocker='rocker')['$(arg sole_shape)']}"/>
   <xacro:if value="${ankle_roll and legacy}"><xacro:ERROR_ankle_roll_needs_a_digitigrade_leg_design/></xacro:if>
   <xacro:property name="hip_drop" value="${0.06 if low else 0.12}"/>
