Commit message: wip: longer digitigrade tail, wedge head and reference details (unvalidated)
Legacy URDF numerically unchanged. MuJoCo/Gazebo revalidation pending.

Co-Authored-By: Claude Opus 5.5 <noreply@anthropic.com>

File: sim/raptor_digitigrade.urdf (robot description, URDF)
Before this commit: robot raptor, 24 links, 23 joints
Links:
- link tail_link: geometry collision box size=0.95 0.065 0.065; visual box size=0.95 0.065 0.065

File: src/raptor_description/urdf/raptor.urdf.xacro (robot description, xacro)
@@ -24,4 +24,9 @@
   <!-- Legacy inertias are the original literals; digitigrade uses the box formula. -->
   <xacro:property name="thigh_ixx" value="${0.0140 if legacy else 1.5*(0.10**2+thigh_length**2)/12}"/>
+  <!-- Tail link: legacy 0.50 m; digitigrade 0.95 m (longer, slimmer, same 0.8 kg; COM moves ~1 cm aft). -->
+  <xacro:property name="tail_length" value="${0.50 if legacy else 0.95}"/>
+  <xacro:property name="tail_width" value="${0.075 if legacy else 0.065}"/>
+  <xacro:property name="tail_ixx" value="${0.0008 if legacy else 0.8*2*tail_width**2/12}"/>
+  <xacro:property name="tail_iyy" value="${0.0169 if legacy else 0.8*(tail_length**2+tail_width**2)/12}"/>
   <xacro:property name="shin_ixx" value="${0.0089 if legacy else 1.1*(0.085**2+shin_length**2)/12}"/>
   <!-- Legacy thigh/shin meshes fit only the legacy lengths. -->
@@ -611,7 +616,7 @@
     <xacro:unless value="${detailed}"><visual>
       <!-- Pitch 관절에서 뒤쪽으로 0.5m 뻗는 꼬리 -->
-      <origin xyz="-0.25 0 0" rpy="0 0 0"/>
-      <geometry>
-        <box size="0.50 0.075 0.075"/>
+      <origin xyz="${-tail_length/2} 0 0" rpy="0 0 0"/>
+      <geometry>
+        <box size="${tail_length} ${tail_width} ${tail_width}"/>
       </geometry>
       <material name="tail_gray">
@@ -626,19 +631,19 @@
     </xacro:if>
     <collision>
-      <origin xyz="-0.25 0 0" rpy="0 0 0"/>
-      <geometry>
-        <box size="0.50 0.075 0.075"/>
-      </geometry>
-    </collision>
-    <inertial>
-      <origin xyz="-0.25 0 0" rpy="0 0 0"/>
+      <origin xyz="${-tail_length/2} 0 0" rpy="0 0 0"/>
+      <geometry>
+        <box size="${tail_length} ${tail_width} ${tail_width}"/>
+      </geometry>
+    </collision>
+    <inertial>
+      <origin xyz="${-tail_length/2} 0 0" rpy="0 0 0"/>
       <mass value="0.8"/>
       <inertia
-        ixx="0.0008"
-        ixy="0.0"
-        ixz="0.0"
-        iyy="0.0169"
-        iyz="0.0"
-        izz="0.0169"/>
+        ixx="${tail_ixx}"
+        ixy="0.0"
+        ixz="0.0"
+        iyy="${tail_iyy}"
+        iyz="0.0"
+        izz="${tail_iyy}"/>
     </inertial>
   </link>
